Commit message: Update robotmctask and motion-control-gateway (#1610)
Co-authored-by: oep <oep@intel.com>

File: libraries/robotics-ai-libraries/motion-control-gateway/humanoid_robot/ti5robot/urdf/ti5.urdf (robot description, URDF)
Before this commit: robot t1, 25 links, 24 joints
Joints:
- joint L_SHOULDER_R: type fixed -> revolute
- joint R_SHOULDER_R: type fixed -> revolute
